Commit message: WIP:  Cheetah Architecture, debugging with RViz, testing new approaches

File: Code/ROS/src/cheetah_ros2/models/THex_Quadruped/model.urdf (robot description, URDF)
Before this commit: robot THex_Quadruped, 13 links, 12 joints
Links:
- added link bl_foot_tip
- added link br_foot_tip
- added link fl_foot_tip
- added link fr_foot_tip
- link base_link: mass None -> 0.30423; geometry collision mesh filename=package://cheetah_ros2/models/THex_Quadruped/meshes/base_li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 scale=1 1 1; visual mesh filename=package://cheetah_ros2/models/THex_Quadruped/meshes/base_li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 scale=1 1 1
- link bl_foot: mass None -> 0.09125; geometry collision mesh filename=package://cheetah_ros2/models/THex_Quadruped/meshes/bl_foot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 scale=1 1 1; visual mesh filename=package://cheetah_ros2/models/THex_Quadruped/meshes/bl_foot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 scale=1 1 1
- link bl_hip: mass None -> 0.14763; geometry collision mesh filename=package://cheetah_ros2/models/THex_Quadruped/meshes/bl_hip_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 scale=1 1 1; visual mesh filename=package://cheetah_ros2/models/THex_Quadruped/meshes/bl_hip.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 scale=1 1 1
- link bl_knee: mass None -> 0.03468; geometry collision mesh filename=package://cheetah_ros2/models/THex_Quadruped/meshes/bl_knee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 scale=1 1 1; visual mesh filename=package://cheetah_ros2/models/THex_Quadruped/meshes/bl_knee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 scale=1 1 1
- link br_foot: mass None -> 0.09125; geometry collision mesh filename=package://cheetah_ros2/models/THex_Quadruped/meshes/br_foot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 scale=1 1 1; visual mesh filename=package://cheetah_ros2/models/THex_Quadruped/meshes/br_foot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 scale=1 1 1
- link br_hip: mass None -> 0.14763; geometry collision mesh filename=package://cheetah_ros2/models/THex_Quadruped/meshes/br_hip_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 scale=1 1 1; visual mesh filename=package://cheetah_ros2/models/THex_Quadruped/meshes/br_hip.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 scale=1 1 1
- link br_knee: mass None -> 0.03468; geometry collision mesh filename=package://cheetah_ros2/models/THex_Quadruped/meshes/br_knee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 scale=1 1 1; visual mesh filename=package://cheetah_ros2/models/THex_Quadruped/meshes/br_knee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 scale=1 1 1
- link fl_foot: mass None -> 0.09125; geometry collision mesh filename=package://cheetah_ros2/models/THex_Quadruped/meshes/fl_foot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 scale=1 1 1; visual mesh filename=package://cheetah_ros2/models/THex_Quadruped/meshes/fl_foot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 scale=1 1 1
- link fl_hip: mass None -> 0.14763; geometry collision mesh filename=package://cheetah_ros2/models/THex_Quadruped/meshes/fl_hip_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 scale=1 1 1; visual mesh filename=package://cheetah_ros2/models/THex_Quadruped/meshes/fl_hip.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 scale=1 1 1
- link fl_knee: mass None -> 0.034681; geometry collision mesh filename=package://cheetah_ros2/models/THex_Quadruped/meshes/fl_knee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 scale=1 1 1; visual mesh filename=package://cheetah_ros2/models/THex_Quadruped/meshes/fl_knee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 scale=1 1 1
- link fr_foot: mass None -> 0.09125; geometry collision mesh filename=package://cheetah_ros2/models/THex_Quadruped/meshes/fr_foot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 scale=1 1 1; visual mesh filename=package://cheetah_ros2/models/THex_Quadruped/meshes/fr_foot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 scale=1 1 1
- link fr_hip: mass None -> 0.14763; geometry collision mesh filename=package://cheetah_ros2/models/THex_Quadruped/meshes/fr_hip_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 scale=1 1 1; visual mesh filename=package://cheetah_ros2/models/THex_Quadruped/meshes/fr_hip.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 scale=1 1 1
- link fr_knee: mass None -> 0.03468; geometry collision mesh filename=package://cheetah_ros2/models/THex_Quadruped/meshes/fr_knee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 scale=1 1 1; visual mesh filename=package://cheetah_ros2/models/THex_Quadruped/meshes/fr_knee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 scale=1 1 1
Joints:
- added joint bl_foot_tip_joint: type fixed, parent bl_foot, child bl_foot_tip, origin xyz=0.09265 0 0 rpy=0 0 0
- added joint br_foot_tip_joint: type fixed, parent br_foot, child br_foot_tip, origin xyz=0.09265 0 0 rpy=0 0 0
- added joint fl_foot_tip_joint: type fixed, parent fl_foot, child fl_foot_tip, origin xyz=0.09265 0 0 rpy=0 0 0
- added joint fr_foot_tip_joint: type fixed, parent fr_foot, child fr_foot_tip, origin xyz=0.09265 0 0 rpy=0 0 0
- joint bl_foot_joint: axis (none) -> 1.11022e-16 -2.35926e-33 1; limit lower=-1.5707 upper=1.5707 effort=0.94140000000000001 velocity=5.2300000000000004 -> lower=-1.5707 upper=1.5707 effort=0.9414 velocity=5.23; origin (none) -> xyz=0.073069 0.018656 -0.00019751 rpy=3.134 0.0073895 0.7853
- joint bl_hip_joint: axis (none) -> 0 0 1; limit lower=-0.7853 upper=0.7853 effort=0.94140000000000001 velocity=5.2300000000000004 -> lower=-0.7853 upper=0.7853 effort=0.9414 velocity=5.23; origin (none) -> xyz=-0.053162 -0.12711 0 rpy=0 0 -2.372
- joint bl_knee_joint: axis (none) -> -5.55112e-17 0 1; limit lower=-1.5707 upper=1.5707 effort=0.94140000000000001 velocity=5.2300000000000004 -> lower=-1.5707 upper=1.5707 effort=0.9414 velocity=5.23; origin (none) -> xyz=0.028451 6.245e-17 0 rpy=-1.5602 0 0
- joint br_foot_joint: axis (none) -> 1.77809e-17 4.33681e-19 1; limit lower=-1.5707 upper=1.5707 effort=0.94140000000000001 velocity=5.2300000000000004 -> lower=-1.5707 upper=1.5707 effort=0.9414 velocity=5.23; origin (none) -> xyz=0.073065 -0.018656 -0.0001221 rpy=-3.1369 0.0045678 -0.7853
- joint br_hip_joint: axis (none) -> 0 0 1; limit lower=-0.7853 upper=0.7853 effort=0.94140000000000001 velocity=5.2300000000000004 -> lower=-0.7853 upper=0.7853 effort=0.9414 velocity=5.23; origin (none) -> xyz=0.053162 -0.12711 0.0005334 rpy=0 0 -0.77529
- joint br_knee_joint: axis (none) -> -1.66533e-16 4.62223e-33 1; limit lower=-1.5707 upper=1.5707 effort=0.94140000000000001 velocity=5.2300000000000004 -> lower=-1.5707 upper=1.5707 effort=0.9414 velocity=5.23; origin (none) -> xyz=0.028449 -6.93889e-18 -1.0842e-19 rpy=1.5643 -0 0
- joint fl_foot_joint: axis (none) -> -4.59702e-17 1.27593e-33 1; limit lower=-1.5707 upper=1.5707 effort=0.94140000000000001 velocity=5.2300000000000004 -> lower=-1.5707 upper=1.5707 effort=0.9414 velocity=5.23; origin (none) -> xyz=0.073066 0.018656 0.00012569 rpy=-3.1368 -0.0047025 0.7853
- joint fl_hip_joint: axis (none) -> 0 0 1; limit lower=-0.7853 upper=0.7853 effort=0.94140000000000001 velocity=5.2300000000000004 -> lower=-0.7853 upper=0.7853 effort=0.9414 velocity=5.23; origin (none) -> xyz=-0.059512 0.078854 0 rpy=0 -0 2.3666
- joint fl_knee_joint: axis (none) -> -5.55112e-17 0 1; limit lower=-1.5707 upper=1.5707 effort=0.94140000000000001 velocity=5.2300000000000004 -> lower=-1.5707 upper=1.5707 effort=0.9414 velocity=5.23; origin (none) -> xyz=0.028449 -6.93889e-18 0 rpy=-1.5775 3.93837e-17 3.91205e-17
- joint fr_foot_joint: axis (none) -> 0 0 1; limit lower=-1.5707 upper=1.5707 effort=0.94140000000000001 velocity=5.2300000000000004 -> lower=-1.5707 upper=1.5707 effort=0.9414 velocity=5.23; origin (none) -> xyz=0.07307 -0.018656 0.0002011 rpy=3.1339 -0.0075232 -0.7853
- joint fr_hip_joint: axis (none) -> 0 0 1; limit lower=-0.7853 upper=0.7853 effort=0.94140000000000001 velocity=5.2300000000000004 -> lower=-0.7853 upper=0.7853 effort=0.9414 velocity=5.23; origin (none) -> xyz=0.059512 0.078854 0.0005334 rpy=0 -0 0.76931
- joint fr_knee_joint: axis (none) -> -5.55112e-17 0 1; limit lower=-1.5707 upper=1.5707 effort=0.94140000000000001 velocity=5.2300000000000004 -> lower=-1.5707 upper=1.5707 effort=0.9414 velocity=5.23; origin (none) -> xyz=0.028451 -6.93889e-18 0 rpy=1.5816 -3.94638e-17 3.90397e-17
