Commit message: Dockerfile: included libraries for posture adaptation. rl_ros2: updated rl_obs, rl_policy, and teleop to allow for all kinds of networks with teleoperation. rlpa_ros2: integrated Zuhair's standalone perception module (WIP)

File: Code/ROS/src/rlpa_ros2/models/THex_Quadruped/model_sim.urdf (robot description, URDF)
Before this commit: robot THex_Quadruped, 13 links, 12 joints
Links:
- added link camera_link, mass 0.001; visual box size=0.04 0.08 0.03
- link base_link: geometry collision mesh filename=package://rlpa_ros2/models/THex_Quadruped/meshes/base_link_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 scale=1 1 1; visual mesh filename=package://rlpa_ros2/models/THex_Quadruped/meshes/base_link.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 scale=1 1 1
- link bl_foot: geometry collision mesh filename=package://rlpa_ros2/models/THex_Quadruped/meshes/bl_foot_co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 scale=1 1 1; visual mesh filename=package://rlpa_ros2/models/THex_Quadruped/meshes/bl_foot.STL scale=1 1 1
- link bl_hip: geometry collision mesh filename=package://rlpa_ros2/models/THex_Quadruped/meshes/bl_hip_col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 scale=1 1 1; visual mesh filename=package://rlpa_ros2/models/THex_Quadruped/meshes/bl_hip.STL scale=1 1 1
- link bl_knee: geometry collision mesh filename=package://rlpa_ros2/models/THex_Quadruped/meshes/bl_knee_co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 scale=1 1 1; visual mesh filename=package://rlpa_ros2/models/THex_Quadruped/meshes/bl_knee.STL scale=1 1 1
- link br_foot: geometry collision mesh filename=package://rlpa_ros2/models/THex_Quadruped/meshes/br_foot_co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 scale=1 1 1; visual mesh filename=package://rlpa_ros2/models/THex_Quadruped/meshes/br_foot.STL scale=1 1 1
- link br_hip: geometry collision mesh filename=package://rlpa_ros2/models/THex_Quadruped/meshes/br_hip_col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 scale=1 1 1; visual mesh filename=package://rlpa_ros2/models/THex_Quadruped/meshes/br_hip.STL scale=1 1 1
- link br_knee: geometry collision mesh filename=package://rlpa_ros2/models/THex_Quadruped/meshes/br_knee_co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 scale=1 1 1; visual mesh filename=package://rlpa_ros2/models/THex_Quadruped/meshes/br_knee.STL scale=1 1 1
- link fl_foot: geometry collision mesh filename=package://rlpa_ros2/models/THex_Quadruped/meshes/fl_foot_co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 scale=1 1 1; visual mesh filename=package://rlpa_ros2/models/THex_Quadruped/meshes/fl_foot.STL scale=1 1 1
- link fl_hip: geometry collision mesh filename=package://rlpa_ros2/models/THex_Quadruped/meshes/fl_hip_col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 scale=1 1 1; visual mesh filename=package://rlpa_ros2/models/THex_Quadruped/meshes/fl_hip.STL scale=1 1 1
- link fl_knee: geometry collision mesh filename=package://rlpa_ros2/models/THex_Quadruped/meshes/fl_knee_co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 scale=1 1 1; visual mesh filename=package://rlpa_ros2/models/THex_Quadruped/meshes/fl_knee.STL scale=1 1 1
- link fr_foot: geometry collision mesh filename=package://rlpa_ros2/models/THex_Quadruped/meshes/fr_foot_co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 scale=1 1 1; visual mesh filename=package://rlpa_ros2/models/THex_Quadruped/meshes/fr_foot.STL scale=1 1 1
- link fr_hip: geometry collision mesh filename=package://rlpa_ros2/models/THex_Quadruped/meshes/fr_hip_col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 scale=1 1 1; visual mesh filename=package://rlpa_ros2/models/THex_Quadruped/meshes/fr_hip.STL scale=1 1 1
- link fr_knee: geometry collision mesh filename=package://rlpa_ros2/models/THex_Quadruped/meshes/fr_knee_co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 scale=1 1 1; visual mesh filename=package://rlpa_ros2/models/THex_Quadruped/meshes/fr_knee.STL scale=1 1 1
Joints:
- added joint camera_joint: type fixed, parent base_link, child camera_link, origin xyz=0.0 0.05 0.15 rpy=0 0.0 1.5708

Commit message: rlpa_ros2: add flat_cave, remove apf, fix point cloud handling

File: Code/ROS/src/rlpa_ros2/models/THex_Quadruped/model_sim.urdf (robot description, URDF)
Before this commit: robot THex_Quadruped, 14 links, 13 joints
Links:
- link camera_link: geometry visual box size=0.01 0.01 0.04
Joints:
- joint camera_joint: origin xyz=0.0 0.05 0.15 rpy=0 0.0 1.5708 -> xyz=0.0 0.13 0.06 rpy=1.5708 0.0 1.5708
